File: PCB/BSF-Control-V1.0/BSF-Control-V1.0.kicad_pcb (KiCad board)
At the start: 2 copper layers, 73.5 x 77 mm, 18 parts, among them J1 I2C Conn 1, J10 Switch, J2 I2C Conn 2, J3 I2C Conn 3, J4 Relay 1, J5 Relay 2, J6 Relay 3, J7 Relay 4, J8 Barrel_Jack_MountingPin, J9 Humidifire Control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

Commit message: Update
Routing:
- net I2C_SCL: track 109.3 -> 108.4 mm
Changed lines of the file:
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@@
 			(outputformat 1)
 			(mirror no)
-			(drillshape 1)
+			(drillshape 0)
 			(scaleselection 1)
-			(outputdirectory "")
+			(outputdirectory "Gerber")
 		)
 	)
@@
 		(tags "connector Molex SL vertical")
 		(property "Reference" "J1"
-			(at 3.81 -3.75 360)
+			(at 3.81 -3.75 0)
 			(layer "F.SilkS")
 			(effects
@@
 		)
 		(property "Value" "I2C Conn 1"
-			(at 3.81 5.25 360)
+			(at 3.81 5.25 0)
 			(layer "F.Fab")
 			(effects
@@
 		)
 		(property "Footprint" "Connector_Molex:Molex_SL_171971-0004_1x04_P2.54mm_Vertical"
-			(at 0 0 360)
+			(at 0 0 0)
 			(layer "F.Fab")
 			(hide yes)
@@
 		)
 		(property "Datasheet" ""
-			(at 0 0 360)
+			(at 0 0 0)
 			(layer "F.Fab")
 			(hide yes)
@@
 		)
 		(property "Description" "Generic connector, single row, 01x04, script generated"
-			(at 0 0 360)
+			(at 0 0 0)
 			(layer "F.Fab")
 			(hide yes)
@@
 		)
 		(fp_text user "${REFERENCE}"
-			(at 3.81 1.85 360)
+			(at 3.81 1.85 0)
 			(layer "F.Fab")
 			(effects
@@
 		)
 		(fp_text user "${REFERENCE}"
-			(at 0 1.27 360)
+			(at 0 1.27 0)
 			(layer "F.Fab")
 			(effects
@@
 		(tags "connector Molex SL vertical")
 		(property "Reference" "J7"
-			(at 6.35 -3.75 360)
+			(at 6.35 -3.75 0)
 			(layer "F.SilkS")
 			(effects
@@
 		)
 		(property "Value" "Relay 4"
-			(at 6.35 5.25 360)
+			(at 6.35 5.25 0)
 			(layer "F.Fab")
 			(effects
@@
 		)
 		(property "Footprint" "Connector_Molex:Molex_SL_171971-0006_1x06_P2.54mm_Vertical"
-			(at 0 0 360)
+			(at 0 0 0)
 			(layer "F.Fab")
 			(hide yes)
@@
 		)
 		(property "Datasheet" ""
-			(at 0 0 360)
+			(at 0 0 0)
 			(layer "F.Fab")
 			(hide yes)
@@
 		)
 		(property "Description" "Generic connector, single row, 01x06, script generated"
-			(at 0 0 360)
+			(at 0 0 0)
 			(layer "F.Fab")
 			(hide yes)
@@
 		)
 		(fp_text user "${REFERENCE}"
-			(at 6.35 1.85 360)
+			(at 6.35 1.85 0)
 			(layer "F.Fab")
 			(effects
@@
 	)
 	(segment
-		(start 147.69 44.19)
-		(end 141 44.19)
+		(start 139.19 44.19)
+		(end 137.5 44.19)
 		(width 0.6)
 		(layer "F.Cu")
@@
 	)
 	(segment
-		(start 139.19 44.19)
-		(end 137.5 44.19)
+		(start 140 44.19)
+		(end 139.19 44.19)
 		(width 0.6)
 		(layer "F.Cu")
@@
 	)
 	(segment
-		(start 140 44.19)
-		(end 139.19 44.19)
+		(start 148.1175 54.2)
+		(end 148.1175 46.1175)
 		(width 0.6)
 		(layer "F.Cu")
@@
 	)
 	(segment
-		(start 148.1175 54.2)
-		(end 148.1175 44.6175)
+		(start 148.1175 46.1175)
+		(end 146.19 44.19)
 		(width 0.6)
 		(layer "F.Cu")
@@
 	)
 	(segment
-		(start 148.1175 44.6175)
-		(end 147.69 44.19)
-		(width 0.6)
-		(layer "F.Cu")
-		(net 4)
-	)
-	(segment
 		(start 140.5 45.5)
 		(end 140.5 44.69)
@@
 	)
 	(segment
+		(start 146.19 44.19)
+		(end 141 44.19)
+		(width 0.6)
+		(layer "F.Cu")
+		(net 4)
+	)
+	(segment
 		(start 125.5 54.54)
 		(end 121.96 54.54)
@@
 	)
 	(segment
-		(start 155.94 82.56)
-		(end 156.5 82)
+		(start 162.5 59)
+		(end 162.5 63.5)
 		(width 0.6)
 		(layer "B.Cu")
@@
 	)
 	(segment
-		(start 156.5 82)
-		(end 156.5 59.25)
+		(start 161 57.5)
+		(end 162.5 59)
 		(width 0.6)
 		(layer "B.Cu")
@@
 	)
 	(segment
-		(start 162.5 63.5)
-		(end 166.96 67.96)
+		(start 158.25 57.5)
+		(end 161 57.5)
 		(width 0.6)
 		(layer "B.Cu")
@@
 	)
 	(segment
-		(start 156.5 59.25)
-		(end 158.25 57.5)
+		(start 162.5 63.5)
+		(end 166.96 67.96)
 		(width 0.6)
 		(layer "B.Cu")
@@
 	)
 	(segment
-		(start 141.9075 82.56)
-		(end 155.94 82.56)
+		(start 156.5 82)
+		(end 156.5 59.25)
 		(width 0.6)
 		(layer "B.Cu")
@@
 	)
 	(segment
-		(start 158.25 57.5)
-		(end 161.5 57.5)
+		(start 155.94 82.56)
+		(end 156.5 82)
 		(width 0.6)
 		(layer "B.Cu")
@@
 	)
 	(segment
-		(start 162.5 58.5)
-		(end 162.5 63.5)
+		(start 141.9075 82.56)
+		(end 155.94 82.56)
 		(width 0.6)
 		(layer "B.Cu")
@@
 	)
 	(segment
-		(start 161.5 57.5)
-		(end 162.5 58.5)
+		(start 156.5 59.25)
+		(end 158.25 57.5)
 		(width 0.6)
 		(layer "B.Cu")
@@
 	)
 	(segment
-		(start 157 86.5)
-		(end 157.5 87)
-		(width 0.6)
-		(layer "F.Cu")
-		(net 21)
-	)
-	(segment
-		(start 159.3475 77.5)
-		(end 158 77.5)
+		(start 158 77.5)
+		(end 156.5 79)
 		(width 0.6)
 		(layer "F.Cu")
@@
 	)
 	(segment
-		(start 157.42 87.08)
-		(end 157.42 91)
+		(start 157.42 86.92)
+		(end 156.5 86)
 		(width 0.6)
 		(layer "F.Cu")
@@
 	)
 	(segment
-		(start 157.5 87)
-		(end 157.42 87.08)
+		(start 156.5 79)
+		(end 156.5 86)
 		(width 0.6)
 		(layer "F.Cu")
@@
 	)
 	(segment
-		(start 158 77.5)
-		(end 157 78.5)
+		(start 157.42 91)
+		(end 157.42 86.92)
 		(width 0.6)
 		(layer "F.Cu")
@@
 	)
 	(segment
-		(start 157 78.5)
-		(end 157 86.5)
+		(start 159.3475 77.5)
+		(end 158 77.5)
 		(width 0.6)
 		(layer "F.Cu")
